Commit message: add gmapping

File: dashgo_description/urdf/dashgobase/dashgobase.xacro (robot description, xacro)
@@ -18,5 +18,5 @@
 -->
  <joint name="laser" type="fixed">
-    <origin xyz="0.00 0.00 0.20" rpy="0 0 0" />
+    <origin xyz="0.15 0.00 0.20" rpy="0 0 0" />
     <parent link="base_link" />
     <child link="base_laser_link" />

Commit message: add gmapping and move_base

File: dashgo_description/urdf/dashgobase/dashgobase.xacro (robot description, xacro)
@@ -17,4 +17,5 @@
    </torso>
 -->
+<!--
  <joint name="laser" type="fixed">
     <origin xyz="0.15 0.00 0.20" rpy="0 0 0" />
@@ -37,3 +38,18 @@
     </inertial>
   </link>
+-->
+  <link name="front_flag">
+      <visual>
+        <origin xyz="0 0 0" rpy="0 0 0" />
+        <geometry>
+          <box size="0.05 0.05 0.001" />
+        </geometry>
+        <material name="TransparentGreen" />
+      </visual>
+  </link>
+  <joint name="front_point_flag" type="fixed">
+    <origin xyz="0.2 0 ${base_length/2}" rpy="0 0 0" />
+    <parent link="base_link"/>
+    <child link="front_flag" />
+  </joint>
 </robot>
